File: circuit/mainBoard_new.brd (EAGLE design)
At the start: 50.2 x 52.8 mm, 22 parts

Commit message: .
Parts:
- removed E$12, E$18: (no value), con-lsta2:FE03-1
- removed E$13: TIP 122, con-lstb:MA03-1
- removed E$15, E$16, E$3, E$4: (no value), con-lsta2:FE01-1
- removed E$2, E$9: (no value), wirepad:2,15/1,0
- removed E$20: 1k, eagle-ltspice:0204/7
- removed E$7: (no value), con-lumberg:1503_09
- moved E$10 37.6 mm to (48.0, 61.1)
- moved E$6 32.6 mm to (41.0, 81.0)
- moved E$5 31.0 mm to (57.8, 70.6)
- moved E$42 30.1 mm to (41.6, 71.5)
- moved E$43 30.1 mm to (62.6, 74.0)
- moved E$1 29.5 mm to (41.0, 61.0)
- moved E$11 25.0 mm to (47.0, 80.9)
- moved E$45 21.0 mm to (55.5, 63.8), turned to 270 degrees
Connections:
- removed net S$10: E$18.5, E$7.2
- removed net S$11: E$13.3, E$20.1
- removed net S$13: E$12.1, E$4.1
- removed net S$16: E$42.4, E$45.2
- removed net S$8: E$11.1, E$18.1
- net S$14: now also E$11.1, E$45.4, E$5.2, E$6.1; no longer E$13.2, E$42.3
- net S$15: now also E$1.1; no longer E$3.1, E$7.3
- net S$2: now also E$42.3, E$45.5; no longer E$16.1, E$45.3
- net S$3: now also E$42.4, E$45.2; no longer E$42.5, E$45.5
- net S$4: now also E$10.1, E$45.3; no longer E$11.2, E$12.2, E$13.1, E$45.4, E$5.2, E$7.1
- net S$5: now also E$42.5; no longer E$20.2
- net S$9: now also E$11.2; no longer E$18.2
Routing:
- net S$14: track 0.00 -> 65.7 mm
- net S$5: track 0.00 -> 57.1 mm
- net S$15: track 0.00 -> 44.5 mm
- net S$2: track 0.00 -> 38.5 mm
- net S$9: track 0.00 -> 29.4 mm
- net S$3: track 0.00 -> 17.8 mm
- net S$4: track 0.00 -> 5.31 mm
Other:
- board outline removed
- board text removed: "0 out"
- board text removed: "5.1 out"
- board text removed: "B+"
- board text removed: "B-"
- board text removed: "G"
- board text removed: "S"
- board text removed: "V"
- board text removed: "b"
- board text removed: "c"
- board text removed: "e"
- board text removed: "switch tilt or external interrupt"

Commit message: da cantina ubuntu
Parts:
- removed E$17: (no value), wirepad:2,15/1,0
- moved E$14 54.0 mm to (59.2, 70.5)
- moved E$8 49.8 mm to (56.6, 70.5)
Routing:
- net S$2: track 38.5 -> 39.6 mm
- net S$5: track 57.1 -> 57.8 mm
Other:
- board outline added: 30 x 31.5 mm
- board text removed: "switch on off"
